File: hardware/fire_alarm/indicators.kicad_sch (KiCad schematic)
At the start: 3 parts, among them Q3 SI2302DS 20V 2.9A

Commit message: feat: complete schematic
Signed-off-by: Trung Hieu Nguyen <hieu.nguyenarc03@gmail.com>
Parts:
- removed D4: LED_Dual_AKAK, LED_SMD:LED_Kingbright_AAA3528ESGCT, symbol Device:LED_Dual_AKAK
- added D5: LED GREEN, LED_THT:LED_D5.0mm, symbol Device:LED
- added D6: LED RED, LED_THT:LED_D5.0mm, symbol Device:LED
- added R19: 33Ohm 0.1W, Resistor_SMD:R_0603_1608Metric_Pad0.98x0.95mm_HandSolder, symbol Device:R
- added R20: 120Ohm 0.1W, Resistor_SMD:R_0603_1608Metric_Pad0.98x0.95mm_HandSolder, symbol Device:R
Connections:
- net GND: now also D5.1 (K)
- new net: D5.2 (A), R19.2
- new net: D6.2 (A), R20.1
- new net +3.3V: R20.2
- new net LED_ALARM: D6.1 (K), R19.1
Other:
- moved on the sheet: BZ1, Q3
