File: hardware/fire_alarm/power.kicad_sch (KiCad schematic)
At the start: 22 parts, among them J1 Barrel_Jack_Switch, U1 MP1584EN-LF-Z, U2 MCP1700x-330xxTT

Commit message: feat: complete schematic
Signed-off-by: Trung Hieu Nguyen <hieu.nguyenarc03@gmail.com>
Parts:
- R15: value 680Ohm 0.1W -> 330Ohm 0.1W
- R16: value 680Ohm 0.1W -> 33Ohm 0.1W
Changed lines of the file:
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@@
 			)
 		)
-		(property "Value" "680Ohm 0.1W"
+		(property "Value" "330Ohm 0.1W"
 			(at 247.65 74.9299 0)
 			(effects
@@
 			)
 		)
-		(property "Value" "680Ohm 0.1W"
+		(property "Value" "33Ohm 0.1W"
 			(at 176.53 133.3499 0)
 			(effects
